File: src/Flight-Computer-Lite/Sheet2.kicad_sch (KiCad schematic)
At the start: 10 parts, among them P4 1984659, U3 SST25VF040B-50-4I-S2AE-T

Commit message: created rev2 schematic
Parts:
- removed B2: PTS647SM38SMTR2LFS, Flight-Computer-Lite:PTS647SM38SMTR2LFS, symbol Flight-Computer:PTS647SM38SMTR2LFS
- removed C16: 0.1uF, Flight-Computer-Lite:CAP_0603, symbol Flight-Computer:CAP_0603
- removed P4: 1984659, Flight-Computer-Lite:1984659, symbol Flight-Computer:1984659
- removed Q?: 2N7002W-7-F, Flight-Computer-Lite:QS5U17TR, symbol Flight-Computer-Lite:2N7002W-7-F
- removed R10, R11, R15, R7: 10k, Flight-Computer-Lite:RES_0603, symbol Flight-Computer:RES_0603
- removed U3: SST25VF040B-50-4I-S2AE-T, Flight-Computer-Lite:SST25VF040B-50-4I-S2AE-T, symbol Flight-Computer:SST25VF040B-50-4I-S2AE-T
- added B1: PTS647SM38SMTR2LFS, Flight-Computer-Lite:PTS647SM38SMTR2LFS, symbol Flight-Computer:PTS647SM38SMTR2LFS
- added C14: 0.1uF, Flight-Computer-Lite:CAP_0603, symbol Flight-Computer:CAP_0603
- added P1: 1984659, Flight-Computer-Lite:1984659, symbol Flight-Computer:1984659
- added Q5, Q6: 2N7002W-7-F, Flight-Computer-Lite:2N7002W-7-F, symbol Flight-Computer-Lite:2N7002W-7-F
- added R17, R18, R19, R20: 10k, Flight-Computer-Lite:RES_0603, symbol Flight-Computer:RES_0603
- added U4: SST25VF040B-50-4I-S2AE-T, Flight-Computer-Lite:SST25VF040B-50-4I-S2AE-T, symbol Flight-Computer:SST25VF040B-50-4I-S2AE-T
Connections:
- net 3.3V: now also R17.2, R18.2, U4.3 (*WP), U4.7 (*HOLD), U4.8 (VDD)
- net BEEP: now also Q6.1 (G); no longer BZ1.1 (-)
- net Earth: now also B1.1, C14.2, Q5.2 (S), Q6.2 (S), R19.1, R20.1, U4.4 (VSS); no longer BZ1.2 (+)
- net FLASH_MISO: now also U4.2 (SO)
- net FLASH_MOSI: now also U4.5 (SI)
- net FLASH_SCK: now also R19.2, U4.6 (SCK)
- net PROG: now also B1.3, C14.1
- net VIN: now also BZ1.1 (-), P1.1 (5)
- net VIN_SW: now also P1.2 (6), Q5.1 (G), R20.2
- net ~{FLASH_SS}: now also R17.1, U4.1 (*CE)
- net ~{SWITCH}: now also Q5.3 (D), R18.1
- new net: BZ1.2 (+), Q6.3 (D)
