File: src/Base-Flight-Computer/Sheet2.kicad_sch (KiCad schematic)
At the start: 9 parts, among them P1 1984659, Q5 2N7002W-7-F, Q6 2N7002W-7-F, U4 SST25VF040B-50-4I-S2AE-T

Commit message: added battery measurement circuit
Parts:
- added R21: 39k, Base-Flight-Computer:RES_0402, symbol Base-Flight-Computer:RES_0402
- added R22: 10k, Base-Flight-Computer:RES_0402, symbol Base-Flight-Computer:RES_0402
- U4: footprint SOIC8_S2A_SST_MCH -> (none)
Connections:
- net Earth: now also R22.1
- net VIN: now also R21.1
- new net VBAT_SENSE: R21.2, R22.2
Other:
- note added: "Battery Voltage Measurement"
Changed lines of the file:
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@@
   (junction (at 83.058 50.292) (diameter 0) (color 0 0 0 0)
   )
+  (junction (at 99.314 101.6) (diameter 0) (color 0 0 0 0)
+  )
   (wire (pts (xy 108.458 70.612) (xy 108.458 71.882))
     (stroke (width 0) (type default))
@@
     (stroke (width 0) (type default))
   )
+  (wire (pts (xy 84.328 101.6) (xy 88.011 101.6))
+    (stroke (width 0) (type default))
+  )
   (wire (pts (xy 84.963 61.722) (xy 83.693 61.722))
     (stroke (width 0) (type default))
@@
     (stroke (width 0) (type default))
   )
+  (wire (pts (xy 99.314 101.6) (xy 101.981 101.6))
+    (stroke (width 0) (type default))
+  )
   (polyline (pts (xy 210.566 82.296) (xy 210.566 133.858))
     (stroke (width 0) (type default))
   )
+  (wire (pts (xy 99.314 112.141) (xy 99.314 114.3))
+    (stroke (width 0) (type default))
+  )
   (polyline (pts (xy 210.185 32.512) (xy 210.185 79.375))
     (stroke (width 0) (type default))
@@
     (stroke (width 0) (type default))
   )
+  (wire (pts (xy 99.314 101.6) (xy 99.314 104.521))
+    (stroke (width 0) (type default))
+  )
+  (wire (pts (xy 95.631 101.6) (xy 99.314 101.6))
+    (stroke (width 0) (type default))
+  )
   (wire (pts (xy 108.458 57.912) (xy 110.998 57.912))
     (stroke (width 0) (type default))
@@
   (wire (pts (xy 106.553 50.292) (xy 110.998 50.292))
     (stroke (width 0) (type default))
+  )
+  (rectangle (start 62.865 82.423) (end 132.08 133.477)
+    (stroke (width 0) (type default))
+    (fill (type none))
+  )
+  (text "Battery Voltage Measurement" (at 74.295 88.265 0)
+    (effects (font (size 2.032 2.032) (thickness 0.4064) bold) (justify left bottom))
   )
   (text "Buzzer" (at 165.735 88.9 0)
@@
     )
   )
+  (global_label "VBAT_SENSE" (shape input) (at 101.981 101.6 0) (fields_autoplaced)
+    (effects (font (size 1.27 1.27)) (justify left))
+    (property "Intersheetrefs" "${INTERSHEET_REFS}" (at 116.3167 101.6 0)
+      (effects (font (size 1.27 1.27)) (justify left) hide)
+    )
+  )
   (global_label "3.3V" (shape input) (at 81.153 40.767 180) (fields_autoplaced)
     (effects (font (size 1.27 1.27)) (justify right))
@@
     (property "Intersheetrefs" "${INTERSHEET_REFS}" (at 199.15 55.0386 0)
       (effects (font (size 1.27 1.27)) (justify left) hide)
+    )
+  )
+  (global_label "VIN" (shape input) (at 84.328 101.6 180) (fields_autoplaced)
+    (effects (font (size 1.27 1.27)) (justify right))
+    (property "Intersheetrefs" "${INTERSHEET_REFS}" (at 78.98 101.5206 0)
+      (effects (font (size 1.27 1.27)) (justify right) hide)
     )
   )
@@
         (path "/13f33ffc-3ab1-449a-9be0-c2c7f72f3b48/f45e6aa6-d67e-481b-8dba-bf06dba939fd"
           (reference "#PWR032") (unit 1)
+        )
+      )
+    )
+  )
+  (symbol (lib_id "Base-Flight-Computer:RES_0402") (at 99.314 108.331 90) (unit 1)
+    (in_bom yes) (on_board yes) (dnp no) (fields_autoplaced)
+    (property "Reference" "R22" (at 101.0666 107.6873 90)
+      (effects (font (size 1.27 1.27)) (justify right))
+    )
+    (property "Value" "10k" (at 101.0666 109.6083 90)
+      (effects (font (size 1.27 1.27)) (justify right))
+    )
+    (property "Footprint" "Base-Flight-Computer:RES_0402" (at 112.014 107.061 0)
+      (effects (font (size 1.27 1.27)) (justify left bottom) hide)
+    )
+    (property "Datasheet" "" (at 99.314 108.331 0)
+      (effects (font (size 1.27 1.27)) (justify left bottom) hide)
+    )
+    (pin "1")
+    (pin "2")
+    (instances
+      (project "Base-Flight-Computer"
+        (path "/13f33ffc-3ab1-449a-9be0-c2c7f72f3b48/f45e6aa6-d67e-481b-8dba-bf06dba939fd"
+          (reference "R22") (unit 1)
         )
       )
@@
     )
   )
+  (symbol (lib_id "Base-Flight-Computer:RES_0402") (at 91.821 101.6 0) (unit 1)
+    (in_bom yes) (on_board yes) (dnp no)
+    (property "Reference" "R21" (at 91.821 99.187 0)
+      (effects (font (size 1.27 1.27)))
+    )
+    (property "Value" "39k" (at 91.821 103.886 0)
+      (effects (font (size 1.27 1.27)))
+    )
+    (property "Footprint" "Base-Flight-Computer:RES_0402" (at 93.091 114.3 0)
+      (effects (font (size 1.27 1.27)) (justify left bottom) hide)
+    )
+    (property "Datasheet" "" (at 91.821 101.6 0)
+      (effects (font (size 1.27 1.27)) (justify left bottom) hide)
+    )
+    (pin "1")
+    (pin "2")
+    (instances
+      (project "Base-Flight-Computer"
+        (path "/13f33ffc-3ab1-449a-9be0-c2c7f72f3b48/f45e6aa6-d67e-481b-8dba-bf06dba939fd"
+          (reference "R21") (unit 1)
+        )
+      )
+    )
+  )
   (symbol (lib_id "Base-Flight-Computer:RES_0402") (at 164.338 67.31 90) (unit 1)
     (in_bom yes) (on_board yes) (dnp no) (fields_autoplaced)
@@
         (path "/13f33ffc-3ab1-449a-9be0-c2c7f72f3b48/f45e6aa6-d67e-481b-8dba-bf06dba939fd"
           (reference "Q6") (unit 1)
+        )
+      )
+    )
+  )
+  (symbol (lib_id "Flight-Computer:Earth") (at 99.314 114.3 0) (unit 1)
+    (in_bom yes) (on_board yes) (dnp no) (fields_autoplaced)
+    (property "Reference" "#PWR031" (at 99.314 120.65 0)
+      (effects (font (size 1.27 1.27)) hide)
+    )
+    (property "Value" "Earth" (at 99.314 118.11 0)
+      (effects (font (size 1.27 1.27)) hide)
+    )
+    (property "Footprint" "" (at 99.314 114.3 0)
+      (effects (font (size 1.27 1.27)) hide)
+    )
+    (property "Datasheet" "" (at 99.314 114.3 0)
+      (effects (font (size 1.27 1.27)) hide)
+    )
+    (pin "1")
+    (instances
+      (project "Base-Flight-Computer"
+        (path "/13f33ffc-3ab1-449a-9be0-c2c7f72f3b48/f45e6aa6-d67e-481b-8dba-bf06dba939fd"
+          (reference "#PWR031") (unit 1)
         )
       )
@@
       (effects (font (size 1.524 1.524)) hide)
     )
-    (property "Footprint" "SOIC8_S2A_SST_MCH" (at 96.393 70.612 0)
+    (property "Footprint" "" (at 96.393 70.612 0)
       (effects (font (size 1.524 1.524)) hide)
     )

Commit message: moved all components to single schematic page
Parts:
- removed BZ1: AT-1438-TWT-R, Flight-Computer:AT-1438-TWT-R, symbol Flight-Computer:AT-1438-TWT-R
- removed P1: 1984659, Base-Flight-Computer:1984659, symbol Base-Flight-Computer:284391-6
- removed Q5, Q6: 2N7002W-7-F, Flight-Computer-Lite:QS5U17TR, symbol Flight-Computer-Lite:2N7002W-7-F
- removed R17, R18, R19, R22: 10k, Base-Flight-Computer:RES_0402, symbol Base-Flight-Computer:RES_0402
- removed R20: 100k, Base-Flight-Computer:RES_0402, symbol Base-Flight-Computer:RES_0402
- removed R21: 39k, Base-Flight-Computer:RES_0402, symbol Base-Flight-Computer:RES_0402
- removed U4: SST25VF040B-50-4I-S2AE-T, symbol Flight-Computer:SST25VF040B-50-4I-S2AE-T
Other:
- note removed: "Arming Switch"
- note removed: "Battery Voltage Measurement"
- note removed: "Buzzer"
- note removed: "Flash"
